File: mixJTAG.sch (EAGLE design)
At the start: 58 parts, among them J1 PLUG-A, J2 CON_HEADER_2X08, Q1 NPN, U1 RCLAMP0544M, U10 SRV05-4, U2 93LC56B, U3 FT2232HLLQFP, U4 XC2C32A-6VQ44C, U5 TC2117-800MA, U6 MCP601, U7 SRV05-4, U8 SRV05-4, U9 SRV05-4, X1 12MHz

Commit message: first layout
Parts:
- removed C26: 100n, rcl:C-EUC0805
- removed Q1: NPN, bb_transistor:BCX70SMD
- removed R6, R8: 10k, rcl:R-US_R0805
- removed R7: 2k, rcl:R-US_R0805
- removed R9: 200R, rcl:R-US_R0805
- removed U10: SRV05-4, bb_tvs:SRV05-4
- added J4: (no value), bb_ml:ML20
- added L4: 600R0.5A, others:DO3316P
- added PCB1: PCB_DP_RECTANGLE-50X100, bb_pcb:PCB_DP_RECTANGLE-50X100
- added RA5: 50R, bb_ra:4R-N
- C10, C11, C18, C25: value 100n -> 4.7u; device rcl:C-EUC0805 -> rcl:CPOL-USB/3528-21R
- C17, C21: value 4.7u -> 100n; device rcl:CPOL-USCT3216 -> rcl:C-EUC0805
- C23: value 4.7u -> 100n
- C5, C6: device rcl:CPOL-USCT3216 -> rcl:CPOL-USB/3528-21R
- C8: value (none) -> 100n; device rcl:CPOL-USCT3216 -> rcl:C-EUC0805
- J2: value CON_HEADER_2X08 -> CON_HEADER_1X03-PTH; device bb_pinheader:CON_HEADER_2X08 -> bb_pinheader:CON_HEADER_1X03-PTH
- J3: value (none) -> CON_HEADER_2X08; device bb_ml:ML20 -> bb_pinheader:CON_HEADER_2X08
- R4: value 10k -> 2k
- R5: value 10k -> 200R
- RA1: value 50R -> 10k
- U1: value RCLAMP0544M -> SRV05-4; device bb_tvs:RCLAMP0544M -> bb_tvs:SRV05-4
- U4: value XC2C32A-6VQ44C -> TC2117-800MA; device bb_xc2c32a:XC2C32A-6VQ44C -> bb_ldo:TC2117-800MA
- U5: value TC2117-800MA -> XC2C32A-6VQ44C; device bb_ldo:TC2117-800MA -> bb_xc2c32a:XC2C32A-6VQ44C
- U6: value MCP601 -> SRV05-4; device bb_op:PIN2PIN-SOIC8 -> bb_tvs:SRV05-4
Connections:
- removed net N$7: R8.1, U6.OUT
- removed net N$8: Q1.B, R8.2
- new net VREF: C24.1, C25.+, J2.3, L4.2
- net +1V8: now also C10.+, C13.1, C22.1, C8.1, U5.VDDINT; no longer C10.1, C11.1, C16.1, C8.+, U4.VDDINT
- net +3V3: now also C16.1, C17.1, C18.+, C19.1, C21.1, J2.1, RA1.1, RA1.2, RA1.3, RA1.4, U4.OUT, U5.VDDAUX, U5.VDDIO1; no longer C13.1, C14.1, C18.1, C21.+, C22.1, R4.1, R5.1, R6.1, U4.VDDAUX, U4.VDDIO1, U5.OUT
- net +5V: no longer Q1.C, U6.VDD
- net CPLD_TCK: now also U5.TCK; no longer U4.TCK
- net CPLD_TDI: now also U5.TDI; no longer U4.TDI
- net CPLD_TDO: now also U5.TDO; no longer U4.TDO
- net CPLD_TMS: now also U5.TMS; no longer U4.TMS
- net EECS: now also RA1.5; no longer R6.2
- net EEDATA: now also R4.1; no longer R7.1
- net EESK: now also RA1.6; no longer R5.2
- net GND: now also C10.-, C11.-, C17.2, C18.-, C21.2, C25.-, C8.2, J4.10, J4.12, J4.14, J4.16, J4.18, J4.20, J4.4, J4.6, J4.8, R5.1, U4.GND, U5.GND@0, U5.GND@1, U5.GND@2, U6.GND; no longer C10.2, C11.2, C17.-, C18.2, C21.-, C25.2, C26.2, C8.-, J3.10, J3.12, J3.14, J3.16, J3.18, J3.20, J3.4, J3.6, J3.8, R9.1, U10.GND, U4.GND@0, U4.GND@1, U4.GND@2, U5.GND, U6.VSS
- net GPIOH0: now also U5.IO_23; no longer U4.IO_23
- net GPIOH1: now also U5.IO_22; no longer U4.IO_22
- net GPIOH2: now also U5.IO_21; no longer U4.IO_21
- net GPIOH3: now also U5.IO_20; no longer U4.IO_20
- net GPIOH4: now also U5.IO_19; no longer U4.IO_19
- net GPIOH5: now also U5.IO_18; no longer U4.IO_18
- net GPIOH6: now also U5.IO_17; no longer U4.IO_17
- net GPIOH7: now also U5.IO_16; no longer U4.IO_16
- net GPIOL0: now also U5.IO_27; no longer U4.IO_31
- net GPIOL1: now also U5.IO_26; no longer U4.IO_30
- net GPIOL2: now also U5.IO_25; no longer U4.IO_29
- net GPIOL3: now also U5.IO_24; no longer U4.IO_28
- net IN13: now also J3.10, J4.11, RA4.8; no longer J2.10, J3.11, RA3.8
- net IN14: now also J3.9, RA4.7; no longer J2.9, J3.13, RA3.7
- net IN15: now also J3.12, J4.13, RA4.6; no longer J2.12, RA3.6
- net IN28: now also J3.15, RA5.5; no longer J2.15, RA4.5
- net IN29: now also J3.16, RA5.6; no longer J2.16, RA4.6
- net IN30: now also J3.13, RA5.7; no longer J2.13, RA4.7
- net IN31: now also J3.14, J4.15, RA5.8; no longer J2.14, RA4.8
- net IN32: now also J3.11, RA4.5; no longer J2.11, RA3.5
- net IO0: now also RA2.1, U5.IO_0, U6.IO1; no longer RA1.1, U4.IO_0, U7.IO4
- net IO1: now also RA2.2, U5.IO_1, U6.IO4; no longer RA1.2, U4.IO_1, U7.IO1
- net IO10: now also RA4.3, U5.IO_10, U8.IO3; no longer RA3.3, U4.IO_10
- net IO11: now also RA4.4, U5.IO_11, U8.IO2; no longer RA3.4, U4.IO_11, U9.IO1
- net IO12: now also RA5.1, U5.IO_12, U9.IO1; no longer RA4.1, U10.IO2, U10.IO4, U4.IO_12
- net IO13: now also RA5.2, U5.IO_13, U9.IO4; no longer RA4.2, U10.IO3, U4.IO_13
- net IO14: now also RA5.3, U5.IO_14, U9.IO3; no longer RA4.3, U4.IO_14
- net IO15: now also RA5.4, U5.IO_15, U9.IO2; no longer RA4.4, U10.IO1, U4.IO_15
- net IO2: now also RA2.3, U5.IO_2, U6.IO3; no longer RA1.3, U4.IO_2, U7.IO2
- net IO3: now also RA2.4, U5.IO_3, U6.IO2; no longer RA1.4, U4.IO_3, U7.IO3
- net IO4: now also RA3.1, U5.IO_4, U7.IO1; no longer RA2.1, U4.IO_4, U8.IO4
- net IO5: now also RA3.2, U5.IO_5, U7.IO4; no longer RA2.2, U4.IO_5, U8.IO2, U8.IO3
- net IO6: now also RA3.3, U5.IO_6, U7.IO3; no longer RA2.3, U4.IO_6
- net IO7: now also RA3.4, U5.IO_7, U7.IO2; no longer RA2.4, U4.IO_7, U8.IO1
- net IO8: now also RA4.1, U5.IO_8, U8.IO1; no longer RA3.1, U4.IO_8, U9.IO2, U9.IO4
- net IO9: now also RA4.2, U5.IO_9, U8.IO4; no longer RA3.2, U4.IO_9, U9.IO3
- net N$1: now also U1.IO4; no longer U1.IO2
- net N$13: now also RA1.8; no longer R7.2
- net N$3: now also C11.+, C14.1, U4.IN; no longer C17.+, C19.1, U5.IN
- net N$4: now also J4.1, J4.2, L4.1; no longer J3.1, J3.2
- net N$6: now also R5.2; no longer R9.2
- net OUT10: now also J3.8, J4.9, RA3.6; no longer J2.8, RA2.6
- net OUT11: now also J3.7, RA3.5; no longer J2.7, RA2.5
- net OUT4: now also J3.2, J4.3, RA2.8; no longer J2.2, J3.3, RA1.8
- net OUT5: now also J3.1, RA2.7; no longer J2.1, J3.5, RA1.7
- net OUT6: now also J3.4, J4.5, RA2.6; no longer J2.4, J3.7, RA1.6
- net OUT7: now also J3.3, RA2.5; no longer J2.3, J3.9, RA1.5
- net OUT8: now also J3.6, J4.7, RA3.8; no longer J2.6, J3.15, RA2.8
- net OUT9: now also J3.5, RA3.7; no longer J2.5, RA2.7
- net REF: no longer C25.1, U6.IN+
- net TCK: now also U5.IO_31; no longer U4.IO_27
- net TDI: now also U5.IO_30; no longer U4.IO_26
- net TDO: now also U5.IO_29; no longer U4.IO_25
- net TGT: now also J2.2, U5.VDDIO2; no longer C24.1, C26.1, Q1.E, U4.VDDIO2, U6.IN-
- net TMS: now also U5.IO_28; no longer U4.IO_24
Other:
- moved on the sheet: C13, C14, C15, C16, C19, C22, C23, C24, C9, R4, R5, RA1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

Commit message: change usb pad
Connections:
- net +3V3: now also R5.2; no longer LED1.A
- net GND: now also LED1.C; no longer R5.1
- net N$6: now also LED1.A, R5.1; no longer LED1.C, R5.2
Other:
- moved on the sheet: LED1, R5
Changed lines of the file:
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@@
 <instance part="C23" gate="G$1" x="148.59" y="146.05"/>
 <instance part="GND14" gate="1" x="148.59" y="135.89"/>
-<instance part="LED1" gate="G$1" x="40.64" y="148.59"/>
+<instance part="LED1" gate="G$1" x="40.64" y="135.89"/>
 <instance part="+3V35" gate="G$1" x="40.64" y="156.21"/>
-<instance part="R5" gate="G$1" x="40.64" y="135.89" smashed="yes" rot="R90">
-<attribute name="NAME" x="39.1414" y="132.08" size="1.778" layer="95" rot="R90"/>
-<attribute name="VALUE" x="43.942" y="132.08" size="1.778" layer="96" rot="R90"/>
+<instance part="R5" gate="G$1" x="40.64" y="146.05" smashed="yes" rot="R90">
+<attribute name="NAME" x="39.1414" y="142.24" size="1.778" layer="95" rot="R90"/>
+<attribute name="VALUE" x="43.942" y="142.24" size="1.778" layer="96" rot="R90"/>
 </instance>
 <instance part="GND7" gate="1" x="40.64" y="125.73"/>
@@
 </segment>
 <segment>
-<pinref part="GND7" gate="1" pin="GND"/>
-<pinref part="R5" gate="G$1" pin="1"/>
-<wire x1="40.64" y1="128.27" x2="40.64" y2="130.81" width="0.1524" layer="91"/>
-</segment>
-<segment>
 <pinref part="GND16" gate="1" pin="GND"/>
 <pinref part="C25" gate="G$1" pin="-"/>
@@
 <label x="201.93" y="-3.81" size="1.27" layer="95" rot="R180" xref="yes"/>
 <pinref part="U9" gate="G$1" pin="GND"/>
+</segment>
+<segment>
+<pinref part="GND7" gate="1" pin="GND"/>
+<pinref part="LED1" gate="G$1" pin="C"/>
+<wire x1="40.64" y1="128.27" x2="40.64" y2="130.81" width="0.1524" layer="91"/>
 </segment>
 </net>
@@
 </segment>
 <segment>
-<pinref part="LED1" gate="G$1" pin="A"/>
-<pinref part="+3V35" gate="G$1" pin="+3V3"/>
-<wire x1="40.64" y1="151.13" x2="40.64" y2="153.67" width="0.1524" layer="91"/>
-</segment>
-<segment>
 <pinref part="J2" gate="J" pin="1"/>
 <pinref part="+3V311" gate="G$1" pin="+3V3"/>
 <wire x1="172.72" y1="114.3" x2="172.72" y2="121.92" width="0.1524" layer="91"/>
+</segment>
+<segment>
+<pinref part="R5" gate="G$1" pin="2"/>
+<pinref part="+3V35" gate="G$1" pin="+3V3"/>
+<wire x1="40.64" y1="151.13" x2="40.64" y2="153.67" width="0.1524" layer="91"/>
 </segment>
 </net>
@@
 </segment>
 </net>
-<net name="N$6" class="0">
-<segment>
-<pinref part="R5" gate="G$1" pin="2"/>
-<pinref part="LED1" gate="G$1" pin="C"/>
-<wire x1="40.64" y1="140.97" x2="40.64" y2="143.51" width="0.1524" layer="91"/>
-</segment>
-</net>
 <net name="N$4" class="0">
 <segment>
@@
 </segment>
 </net>
+<net name="N$6" class="0">
+<segment>
+<pinref part="LED1" gate="G$1" pin="A"/>
+<pinref part="R5" gate="G$1" pin="1"/>
+<wire x1="40.64" y1="138.43" x2="40.64" y2="140.97" width="0.1524" layer="91"/>
+</segment>
+</net>
