File: mixJTAG.brd (EAGLE design)
At the start: 100 x 80 mm, 57 parts, among them J1 PLUG-A, J2 CON_HEADER_1X03-PTH, J3 CON_HEADER_2X08, U1 SRV05-4, U2 93LC56B, U3 FT2232HLLQFP, U4 TC2117-800MA, U5 XC2C32A-6VQ44C, U6 SRV05-4, U7 SRV05-4, U8 SRV05-4, U9 SRV05-4, X1 12MHz

Commit message: more via
Routing:
- net GND: track 237.1 -> 75.4 mm, vias 39 -> 42

Commit message: back up committing
Parts:
- L1, L2, L3: device others:R0805 -> rcl:L2012C
- L4: value 600R0.5A -> 600R0.4A; device others:R0805 -> rcl:L2012C

Commit message: add io buffer board
Parts:
- added C26, C28, C29, C30: 100N, rcl:C0805
- added C27: 4.7u, rcl:SMC_A
- added D1: 1N4148DO35-7, diode:DO35-7
- added J10, J11, J12, J13, J5, J6, J8, J9: CON_HEADER_1X08-PTH, bb_pinheader:M1X8
- added J14: CON_HEADER_2X02-PTH, bb_pinheader:M2X2
- added U10, U11, U12, U13: 74244DW, bb_74:SO20W
Connections:
- new net +12V: D1.A, J14.1, J14.2
- new net 0V: C26.2, C27.-, C28.2, C29.2, C30.2, J14.3, J14.4, U10.1, U10.10, U10.19, U11.1, U11.10, U11.19, U12.1, U12.10, U12.19, U13.1, U13.10, U13.19
- new net N$10: J10.5, U10.6
- new net N$11: J10.4, U10.5
- new net N$12: J10.3, U10.4
- new net N$14: J10.2, U10.3
- new net N$15: J10.1, U10.2
- new net N$16: J5.8, U10.11
- new net N$17: J5.7, U10.12
- new net N$18: J5.6, U10.13
- new net N$19: J5.5, U10.14
- new net N$20: J5.4, U10.15
- new net N$21: J5.3, U10.16
- new net N$22: J5.2, U10.17
- new net N$23: J5.1, U10.18
- new net N$24: J11.8, U11.9
- new net N$25: J11.7, U11.8
- new net N$26: J11.6, U11.7
- new net N$27: J11.5, U11.6
- new net N$28: J11.4, U11.5
- new net N$29: J11.3, U11.4
- new net N$30: J11.2, U11.3
- new net N$31: J11.1, U11.2
- new net N$32: J6.8, U11.11
- new net N$33: J6.7, U11.12
- new net N$34: J6.6, U11.13
- new net N$35: J6.5, U11.14
- new net N$36: J6.4, U11.15
- new net N$37: J6.3, U11.16
- new net N$38: J6.2, U11.17
- new net N$39: J6.1, U11.18
- new net N$40: J12.8, U12.9
- new net N$41: J12.7, U12.8
- new net N$42: J12.6, U12.7
- new net N$43: J12.5, U12.6
- new net N$44: J12.4, U12.5
- new net N$45: J12.3, U12.4
- new net N$46: J12.2, U12.3
- new net N$47: J12.1, U12.2
- new net N$48: J8.8, U12.11
- new net N$49: J8.7, U12.12
- new net N$50: J8.6, U12.13
- new net N$51: J8.5, U12.14
- new net N$52: J8.4, U12.15
- new net N$53: J8.3, U12.16
- new net N$54: J8.2, U12.17
- new net N$55: J8.1, U12.18
- new net N$56: J13.8, U13.9
- new net N$57: J13.7, U13.8
- new net N$58: J13.6, U13.7
- new net N$59: J13.5, U13.6
- new net N$60: J13.4, U13.5
- new net N$61: J13.3, U13.4
- new net N$62: J13.2, U13.3
- new net N$63: J13.1, U13.2
- new net N$64: J9.8, U13.11
- new net N$65: J9.7, U13.12
- new net N$66: J9.6, U13.13
- new net N$67: J9.5, U13.14
- new net N$68: J9.4, U13.15
- new net N$69: J9.3, U13.16
- new net N$7: J10.8, U10.9
- new net N$70: J9.2, U13.17
- new net N$71: J9.1, U13.18
- new net N$8: J10.7, U10.8
- new net N$9: J10.6, U10.7
- new net VCC: C26.1, C27.+, C28.1, C29.1, C30.1, D1.C, U10.20, U11.20, U12.20, U13.20
Routing:
- net VCC: track 0.00 -> 87.2 mm
- net +12V: track 0.00 -> 17.6 mm
- net N$71: track 0.00 -> 11.3 mm
- net N$23: track 0.00 -> 11.3 mm
- net N$55: track 0.00 -> 11.3 mm
- net N$39: track 0.00 -> 11.3 mm
- net N$70: track 0.00 -> 10.8 mm
- net N$54: track 0.00 -> 10.8 mm
- net N$38: track 0.00 -> 10.8 mm
- net N$22: track 0.00 -> 10.8 mm
- net N$53: track 0.00 -> 10.3 mm
- net N$32: track 0.00 -> 10.3 mm
- net N$16: track 0.00 -> 10.3 mm
- net N$21: track 0.00 -> 10.3 mm
- net N$69: track 0.00 -> 10.3 mm
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- added copper zone on layer 1, net 0V
- added copper zone on layer 16, net 0V
Other:
- board size 100 x 80 mm -> 100 x 83.8 mm
- board text added: "1 2 3 4 5 6 7 8 9 10 11 12 13 14 15 16 17 18 19 20 21 22 23 24 25 26 27 28 29 30 31 32"
- board text added: "3.3v"
- board text added: "IOBuf"
- board text added: "Vext"
- board text added: "mixJTAG"
- board text added: "v1.0"

Commit message: change to 0805 current limit resistor
Parts:
- removed J14: CON_HEADER_2X02-PTH, bb_pinheader:M2X2
- removed RA1, RA2, RA3, RA4: 50R, bb_ra:EXBV8V
- added J7: CON_HEADER_1X08-PTH, bb_pinheader:M1X8
- added R10, R11, R12, R13, R14, R15, R16, R17, R18, R19, R20, R21, R22, R23, R24, R9: 50R, rcl:R0805
- C26, C28, C29: value 100N -> 100n
- C27: value 4.7u -> 100n; device rcl:SMC_A -> rcl:C0805
- C30: value 100N -> 4.7u; device rcl:C0805 -> rcl:A/3216-18R
- J11: value CON_HEADER_1X08-PTH -> CON_HEADER_2X02-PTH; device bb_pinheader:M1X8 -> bb_pinheader:M2X2
- J4: value (none) -> CON_HEADER_2X10-PTH; device bb_ml:ML20 -> bb_pinheader:M2X10
- L4: value 600R0.4A -> 600R/0.4A
- LED1: value (none) -> RED
- R3, R7: value 2k -> 2K
- R4, R5, R6: value 2k -> 10K
- moved C30 64.8 mm to (11.4, 68.5)
- moved J10 61.0 mm to (85.1, 54.6)
- moved C26 61.0 mm to (76.2, 66.0)
- moved C27 44.5 mm to (55.9, 66.0), turned to 270 degrees
- moved C29 40.6 mm to (15.2, 66.0)
- moved J11 38.4 mm to (6.35, 59.7)
- moved J9 32.5 mm to (64.8, 54.6)
- moved J12 25.4 mm to (64.8, 80.0)
- moved J13 25.4 mm to (85.1, 80.0)
- moved J5 25.4 mm to (24.1, 54.6)
- moved J6 25.4 mm to (44.5, 54.6)
- moved J8 20.3 mm to (44.5, 80.0)
- moved J3 3.56 mm to (85.1, 24.9)
- moved U9 2.68 mm to (71.1, 16.3)
- moved U6 2.56 mm to (71.1, 34.0)
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Connections:
- removed net 0V: C26.2, C27.-, C28.2, C29.2, C30.2, J14.3, J14.4, U10.1, U10.10, U10.19, U11.1, U11.10, U11.19, U12.1, U12.10, U12.19, U13.1, U13.10, U13.19
- new net GNDA: C26.2, C27.2, C28.2, C29.2, C30.-, J11.3, J11.4, U10.1, U10.10, U10.19, U11.1, U11.10, U11.19, U12.1, U12.10, U12.19, U13.1, U13.10, U13.19
- net +12V: now also J11.1, J11.2; no longer J14.1, J14.2
- net IN13: now also R17.2; no longer RA3.8
- net IN14: now also R18.2; no longer RA3.7
- net IN15: now also R19.2; no longer RA3.6
- net IN28: now also R24.2; no longer RA4.5
- net IN29: now also R23.2; no longer RA4.6
- net IN30: now also R22.2; no longer RA4.7
- net IN31: now also R21.2; no longer RA4.8
- net IN32: now also R20.2; no longer RA3.5
- net IO0: now also R9.1, U6.6; no longer RA1.1, U6.1
- net IO1: now also R10.1, U6.1; no longer RA1.2, U6.6
- net IO10: now also R19.1, U8.3; no longer RA3.3, U8.4
- net IO11: now also R20.1, U8.4; no longer RA3.4, U8.3
- net IO12: now also R21.1, U9.6; no longer RA4.1, U9.1
- net IO13: now also R22.1, U9.1; no longer RA4.2, U9.6
- net IO14: now also R23.1, U9.3; no longer RA4.3, U9.4
- net IO15: now also R24.1, U9.4; no longer RA4.4, U9.3
- net IO2: now also R11.1, U6.3; no longer RA1.3, U6.4
- net IO3: now also R12.1, U6.4; no longer RA1.4, U6.3
- net IO4: now also R13.1, U7.6; no longer RA2.1, U7.1
- net IO5: now also R14.1, U7.1; no longer RA2.2, U7.6
- net IO6: now also R15.1, U7.3; no longer RA2.3, U7.4
- net IO7: now also R16.1, U7.4; no longer RA2.4, U7.3
- net IO8: now also R17.1, U8.6; no longer RA3.1, U8.1
- net IO9: now also R18.1, U8.1; no longer RA3.2, U8.6
- net N$10: now also J5.5; no longer J10.5
- net N$11: now also J5.4; no longer J10.4
- net N$12: now also J5.3; no longer J10.3
- net N$14: now also J5.2; no longer J10.2
- net N$15: now also J5.1; no longer J10.1
- net N$16: now also J7.8; no longer J5.8
- net N$17: now also J7.7; no longer J5.7
- net N$18: now also J7.6; no longer J5.6
- net N$19: now also J7.5; no longer J5.5
- net N$20: now also J7.4; no longer J5.4
- net N$21: now also J7.3; no longer J5.3
- net N$22: now also J7.2; no longer J5.2
- net N$23: now also J7.1; no longer J5.1
- net N$24: now also J6.8; no longer J11.8
- net N$25: now also J6.7; no longer J11.7
- net N$26: now also J6.6; no longer J11.6
- net N$27: now also J6.5; no longer J11.5
- net N$28: now also J6.4; no longer J11.4
- net N$29: now also J6.3; no longer J11.3
- net N$30: now also J6.2; no longer J11.2
- net N$31: now also J6.1; no longer J11.1
- net N$32: now also J8.8; no longer J6.8
- net N$33: now also J8.7; no longer J6.7
- net N$34: now also J8.6; no longer J6.6
- net N$35: now also J8.5; no longer J6.5
- net N$36: now also J8.4; no longer J6.4
- net N$37: now also J8.3; no longer J6.3
- net N$38: now also J8.2; no longer J6.2
- net N$39: now also J8.1; no longer J6.1
- net N$40: now also J9.8; no longer J12.8
- net N$41: now also J9.7; no longer J12.7
- net N$42: now also J9.6; no longer J12.6
- net N$43: now also J9.5; no longer J12.5
- net N$44: now also J9.4; no longer J12.4
- net N$45: now also J9.3; no longer J12.3
- net N$46: now also J9.2; no longer J12.2
- net N$47: now also J9.1; no longer J12.1
- net N$48: now also J12.8; no longer J8.8
- net N$49: now also J12.7; no longer J8.7
- net N$50: now also J12.6; no longer J8.6
- net N$51: now also J12.5; no longer J8.5
- net N$52: now also J12.4; no longer J8.4
- net N$53: now also J12.3; no longer J8.3
- net N$54: now also J12.2; no longer J8.2
- net N$55: now also J12.1; no longer J8.1
- net N$56: now also J10.8; no longer J13.8
- net N$57: now also J10.7; no longer J13.7
- net N$58: now also J10.6; no longer J13.6
- net N$59: now also J10.5; no longer J13.5
- net N$60: now also J10.4; no longer J13.4
- net N$61: now also J10.3; no longer J13.3
- net N$62: now also J10.2; no longer J13.2
- net N$63: now also J10.1; no longer J13.1
- net N$64: now also J13.8; no longer J9.8
- net N$65: now also J13.7; no longer J9.7
- net N$66: now also J13.6; no longer J9.6
- net N$67: now also J13.5; no longer J9.5
- net N$68: now also J13.4; no longer J9.4
- net N$69: now also J13.3; no longer J9.3
- net N$7: now also J5.8; no longer J10.8
- net N$70: now also J13.2; no longer J9.2
- net N$71: now also J13.1; no longer J9.1
- net N$8: now also J5.7; no longer J10.7
- net N$9: now also J5.6; no longer J10.6
- net OUT10: now also R15.2; no longer RA2.6
- net OUT11: now also R16.2; no longer RA2.5
- net OUT4: now also R9.2; no longer RA1.8
- net OUT5: now also R10.2; no longer RA1.7
- net OUT6: now also R11.2; no longer RA1.6
- net OUT7: now also R12.2; no longer RA1.5
- net OUT8: now also R13.2; no longer RA2.8
- net OUT9: now also R14.2; no longer RA2.7
- net VCC: now also C27.1, C30.+; no longer C27.+, C30.1
Routing:
- net GNDA: track 0.00 -> 28.1 mm, vias 0 -> 11
- net GND: track 75.4 -> 59.3 mm, vias 42 -> 44
- net IO6: track 16.4 -> 19.6 mm, vias 2 -> 1
- net IO7: track 14.7 -> 17.6 mm
- net IO3: track 16.8 -> 19.7 mm
- net IO14: track 22.0 -> 24.9 mm, vias 2 -> 1
- net IO1: track 23.6 -> 26.3 mm, vias 2 -> 1
- net IO5: track 17.2 -> 19.9 mm, vias 2 -> 1
- net IO10: track 17.3 -> 19.9 mm, vias 2 -> 1
- net IO13: track 20.9 -> 23.4 mm, vias 2 -> 1
- net IO11: track 14.9 -> 17.4 mm
- net IO9: track 16.9 -> 19.2 mm, vias 2 -> 1
- net IO12: track 17.0 -> 19.3 mm
- net N$4: track 11.2 -> 13.5 mm
- net IO15: track 22.0 -> 24.3 mm
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- added copper zone on layer 1, net GNDA
- added copper zone on layer 16, net GNDA
- removed copper zone on layer 1, net 0V
- removed copper zone on layer 16, net 0V

Commit message: more output
Parts:
- moved C9 5.30 mm to (26.7, 17.0), flipped to the bottom, turned to 90 degrees
- moved J10 1.27 mm to (85.1, 55.9)
- moved J11 1.27 mm to (6.35, 61.0)
- moved J5 1.27 mm to (24.1, 55.9)
- moved J6 1.27 mm to (44.5, 55.9)
- moved J9 1.27 mm to (64.8, 55.9)
- moved C26 1.27 mm to (76.2, 67.3)
- moved C27 1.27 mm to (55.9, 67.3)
- moved C28 1.27 mm to (35.6, 67.3)
- moved C29 1.27 mm to (15.2, 67.3)
- moved C30 1.27 mm to (11.4, 69.7)
- moved D1 1.27 mm to (7.62, 72.4)
- moved J12 1.27 mm to (64.8, 81.3)
- moved J13 1.27 mm to (85.1, 81.3)
- moved J7 1.27 mm to (24.1, 81.3)
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Routing:
- net GND: track 59.3 -> 63.2 mm
- net VPLL: track 11.7 -> 12.4 mm
- net +1V8: track 65.2 -> 64.6 mm, vias 4 -> 5
- net !RESET: track 6.85 -> 6.22 mm
Other:
- board size 100 x 83.8 mm -> 100 x 100 mm
- board text added: "VTref nTRST TDI TMS TCK RTCK TDO nSRST DBGRQ DBGACK"
- board text added: "Vsup GND GND GND GND GND GND GND GND GND"
